File: esquemas/cerradura.kicad_sch (KiCad schematic)
At the start: 2 parts, among them J1 Conn_02x20_Odd_Even, J2 Conn_02x20_Odd_Even

Commit message: update
Parts:
- added J3: esp32_c3_right_socket, Connector_Harwin:Harwin_M20-89008xx_1x08_P2.54mm_Horizontal, symbol Connector:Conn_01x08_Socket
- added J4: num_keypad, Connector_Harwin:Harwin_M20-89008xx_1x08_P2.54mm_Horizontal, symbol Connector:Conn_01x08_Socket
- added J5: esp32_c3_left_socket, Connector_Harwin:Harwin_M20-89008xx_1x08_P2.54mm_Horizontal, symbol Connector:Conn_01x08_Socket
- added J6: R305-sensor, Connector:FanPinHeader_1x04_P2.54mm_Vertical, symbol Connector:Conn_01x04_Pin
- added J7: RC522-sensor, Connector_Harwin:Harwin_M20-89008xx_1x08_P2.54mm_Horizontal, symbol Connector:Conn_01x08_Socket
- added J8: ssd1306-dsp, Connector_Harwin:Harwin_M20-89004xx_1x04_P2.54mm_Horizontal, symbol Connector:Conn_01x04_Socket
Connections:
- net +3.3V: now also J3.3 (Pin_3), J7.1 (Pin_1), J8.4 (Pin_4)
- net +5V: now also J6.1 (Pin_1)
- net GND: now also J3.2 (Pin_2), J6.2 (Pin_2), J7.3 (Pin_3), J8.3 (Pin_3)
- net ssd1306_sda: now reaches J2.19 (Pin_19)
- net ssd1306_sda: now also J8.1 (Pin_1)
- net ssd1306_scl: now reaches J2.21 (Pin_21)
- net ssd1306_scl: now also J8.2 (Pin_2)
- net esp32_tx: now reaches J2.23 (Pin_23)
- net esp32_tx: now also J5.8 (Pin_8)
- net esp32_rx: now reaches J2.25 (Pin_25)
- net esp32_rx: now also J5.7 (Pin_7)
- net kp_c1: now reaches J2.31 (Pin_31)
- net kp_c1: now also J4.6 (Pin_6)
- net kp_f0: now reaches J2.33 (Pin_33)
- net kp_c2: now reaches J2.34 (Pin_34)
- net kp_c2: now also J4.7 (Pin_7)
- net kp_f3: now reaches J2.35 (Pin_35)
- net kp_f3: now also J4.4 (Pin_4)
- net kp_f1: now reaches J2.36 (Pin_36)
- net kp_f1: now also J4.2 (Pin_2)
- net kp_f2: now reaches J2.37 (Pin_37)
- net kp_f2: now also J4.3 (Pin_3)
- net kp_c0: now reaches J2.39 (Pin_39)
- net kp_c0: now also J4.5 (Pin_5)
- net rc522-miso: now reaches J1.18 (Pin_18)
- net rc522-miso: now also J7.5 (Pin_5)
- net rc522-sck: now reaches J1.20 (Pin_20)
- net rc522-sck: now also J7.7 (Pin_7)
- net rc522-mosi: now reaches J1.21 (Pin_21)
- net rc522-mosi: now also J7.6 (Pin_6)
- net r305_tx: now reaches J1.31 (Pin_31)
- net r305_tx: now also J6.3 (Pin_3)
- net r305_rx: now reaches J1.32 (Pin_32)
- net r305_rx: now also J6.4 (Pin_4)
- net rc522-ss: now reaches J1.35 (Pin_35)
- net rc522-ss: now also J7.8 (Pin_8)
- net rc522-rst: now reaches J1.38 (Pin_38)
- net rc522-rst: now also J7.2 (Pin_2)
- new net kp_c3: J4.8 (Pin_8)
- new net rc522-irq: J7.4 (Pin_4)
- new net tfil0: J4.1 (Pin_1)

Commit message: update2
Parts:
- added J10: drv882x_righ_socket, Connector_Harwin:Harwin_M20-89008xx_1x08_P2.54mm_Horizontal, symbol Connector:Conn_01x08_Socket
- added J11: 2n2222, Connector_Harwin:Harwin_M20-89003xx_1x03_P2.54mm_Horizontal, symbol Connector:Conn_01x03_Socket
- added J12: buzzer, Connector_AMASS:AMASS_XT30PW-M_1x02_P2.50mm_Horizontal, symbol Connector_Generic:Conn_01x02
- added J9: drv882x_left_socket, Connector_Harwin:Harwin_M20-89008xx_1x08_P2.54mm_Horizontal, symbol Connector:Conn_01x08_Socket
- J6: value R305-sensor -> R305_sensor
- J7: value RC522-sensor -> RC522_sensor
- J8: value ssd1306-dsp -> ssd1306_dsp
Connections:
- net +3.3V: now also J10.3 (Pin_3), J9.5 (Pin_5), J9.6 (Pin_6)
- net +5V: now also J12.1 (Pin_1)
- net GND: now also J10.2 (Pin_2), J10.8 (Pin_8), J11.3 (Pin_3)
- net drv882x_en: now reaches J1.29 (Pin_29)
- net drv882x_en: now also J9.1 (Pin_1)
- net drv882x_step: now reaches J1.33 (Pin_33)
- net drv882x_step: now also J9.7 (Pin_7)
- net buzzer_sgn: now reaches J1.34 (Pin_34)
- net buzzer_sgn: now also J11.2 (Pin_2)
- net drv882x_dir: now reaches J1.40 (Pin_40)
- net drv882x_dir: now also J9.8 (Pin_8)
- new net: J11.1 (Pin_1), J12.2 (Pin_2)
- new net drv882x_a1: J10.6 (Pin_6)
- new net drv882x_a2: J10.7 (Pin_7)
- new net drv882x_b1: J10.5 (Pin_5)
- new net drv882x_b2: J10.4 (Pin_4)

Commit message: update3
Parts:
- removed J12: buzzer, Connector_AMASS:AMASS_XT30PW-M_1x02_P2.50mm_Horizontal, symbol Connector_Generic:Conn_01x02
- added J13: bornes_motor, TerminalBlock:TerminalBlock_Altech_AK300-4_P5.00mm, symbol Connector:Screw_Terminal_01x04
- added J14: bornes_buzzer, TerminalBlock:TerminalBlock_Altech_AK300-2_P5.00mm, symbol Connector:Screw_Terminal_01x02
Connections:
- net +5V: now also J14.1 (Pin_1)
- net drv882x_a1: now also J13.3 (Pin_3)
- net drv882x_a2: now also J13.4 (Pin_4)
- net drv882x_b1: now also J13.2 (Pin_2)
- net drv882x_b2: now also J13.1 (Pin_1)
- net at J11.1 (Pin_1): now also J14.2 (Pin_2)
Changed lines of the file:
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@@
 	(wire
 		(pts
+			(xy 146.05 175.26) (xy 144.78 175.26)
+		)
+		(stroke
+			(width 0)
+			(type default)
+		)
+	)
+	(wire
+		(pts
 			(xy 43.18 163.83) (xy 41.91 163.83)
 		)
@@
 	(wire
 		(pts
+			(xy 146.05 170.18) (xy 144.78 170.18)
+		)
+		(stroke
+			(width 0)
+			(type default)
+		)
+	)
+	(wire
+		(pts
 			(xy 44.45 119.38) (xy 43.18 119.38)
 		)
@@
 	(wire
 		(pts
+			(xy 146.05 167.64) (xy 144.78 167.64)
+		)
+		(stroke
+			(width 0)
+			(type default)
+		)
+	)
+	(wire
+		(pts
 			(xy 31.75 130.81) (xy 34.29 130.81)
 		)
@@
 	(wire
 		(pts
+			(xy 146.05 172.72) (xy 144.78 172.72)
+		)
+		(stroke
+			(width 0)
+			(type default)
+		)
+	)
+	(wire
+		(pts
 			(xy 130.81 123.19) (xy 134.62 123.19)
 		)
@@
 		)
 	)
+	(label "drv882x_b1"
+		(at 144.78 170.18 180)
+		(effects
+			(font
+				(size 1.27 1.27)
+			)
+			(justify right bottom)
+		)
+	)
 	(label "kp_c0"
 		(at 129.54 101.6 180)
@@
 		)
 	)
+	(label "drv882x_a2"
+		(at 144.78 175.26 180)
+		(effects
+			(font
+				(size 1.27 1.27)
+			)
+			(justify right bottom)
+		)
+	)
 	(label "rc522-sck"
 		(at 149.86 125.73 90)
@@
 		)
 	)
+	(label "drv882x_a1"
+		(at 144.78 172.72 180)
+		(effects
+			(font
+				(size 1.27 1.27)
+			)
+			(justify right bottom)
+		)
+	)
 	(label "kp_f0"
 		(at 129.54 93.98 180)
@@
 		)
 	)
+	(label "drv882x_b2"
+		(at 144.78 167.64 180)
+		(effects
+			(font
+				(size 1.27 1.27)
+			)
+			(justify right bottom)
+		)
+	)
 	(label "tfil0"
 		(at 101.6 125.73 90)
@@
 	)
 	(symbol
-		(lib_id "Connector:Conn_01x08_Socket")
-		(at 109.22 132.08 90)
-		(mirror x)
+		(lib_id "Connector:Screw_Terminal_01x04")
+		(at 151.13 170.18 0)
 		(unit 1)
 		(exclude_from_sim no)
@@
 		(on_board yes)
 		(dnp no)
-		(property "Reference" "J4"
-			(at 110.49 137.16 90)
+		(fields_autoplaced yes)
+		(property "Reference" "J13"
+			(at 153.67 170.1799 0)
 			(effects
 				(font
 					(size 1.27 1.27)
 				)
+				(justify left)
 			)
 		)
-		(property "Value" "num_keypad"
-			(at 110.49 134.62 90)
+		(property "Value" "bornes_motor"
+			(at 153.67 172.7199 0)
 			(effects
 				(font
 					(size 1.27 1.27)
 				)
+				(justify left)
 			)
 		)
-		(property "Footprint" "Connector_Harwin:Harwin_M20-89008xx_1x08_P2.54mm_Horizontal"
-			(at 109.22 132.08 0)
+		(property "Footprint" "TerminalBlock:TerminalBlock_Altech_AK300-4_P5.00mm"
+			(at 151.13 170.18 0)
 			(effects
 				(font
@@
 		)
 		(property "Datasheet" "~"
-			(at 109.22 132.08 0)
+			(at 151.13 170.18 0)
 			(effects
 				(font
@@
 			)
 		)
-		(property "Description" "Generic connector, single row, 01x08, script generated"
-			(at 109.22 132.08 0)
+		(property "Description" "Generic screw terminal, single row, 01x04, script generated (kicad-library-utils/schlib/autogen/connector/)"
+			(at 151.13 170.18 0)
 			(effects
 				(font
@@
 			)
 		)
-		(pin "2"
-		)
 		(pin "1"
 		)
 		(pin "3"
 		)
-		(pin "4"
-		)
-		(pin "5"
-		)
-		(pin "8"
-		)
-		(pin "6"
+		(pin "2"
 		)
-		(pin "7"
+		(pin "4"
 		)
 		(instances
 			(project ""
 				(path "/5ec40689-7e61-4c5f-9022-56a5e47f7bec"
-					(reference "J4")
+					(reference "J13")
 					(unit 1)
 				)
@@
 	)
 	(symbol
-		(lib_id "power:+5V")
-		(at 34.29 148.59 0)
+		(lib_id "Connector:Conn_01x08_Socket")
+		(at 109.22 132.08 90)
+		(mirror x)
 		(unit 1)
 		(exclude_from_sim no)
@@
 		(on_board yes)
 		(dnp no)
-		(property "Reference" "#PWR017"
-			(at 34.29 152.4 0)
+		(property "Reference" "J4"
+			(at 110.49 137.16 90)
 			(effects
 				(font
 					(size 1.27 1.27)
 				)
-				(hide yes)
 			)
 		)
-		(property "Value" "+5V"
-			(at 34.29 143.51 0)
+		(property "Value" "num_keypad"
+			(at 110.49 134.62 90)
 			(effects
 				(font
@@
 			)
 		)
-		(property "Footprint" ""
-			(at 34.29 148.59 0)
+		(property "Footprint" "Connector_Harwin:Harwin_M20-89008xx_1x08_P2.54mm_Horizontal"
+			(at 109.22 132.08 0)
 			(effects
 				(font
@@
 			)
 		)
-		(property "Datasheet" ""
-			(at 34.29 148.59 0)
+		(property "Datasheet" "~"
+			(at 109.22 132.08 0)
 			(effects
 				(font
@@
 			)
 		)
-		(property "Description" "Power symbol creates a global label with name \"+5V\""
-			(at 34.29 148.59 0)
+		(property "Description" "Generic connector, single row, 01x08, script generated"
+			(at 109.22 132.08 0)
 			(effects
 				(font
@@
 			)
 		)
+		(pin "2"
+		)
 		(pin "1"
 		)
+		(pin "3"
+		)
+		(pin "4"
+		)
+		(pin "5"
+		)
+		(pin "8"
+		)
+		(pin "6"
+		)
+		(pin "7"
+		)
 		(instances
-			(project "cerradura"
+			(project ""
 				(path "/5ec40689-7e61-4c5f-9022-56a5e47f7bec"
-					(reference "#PWR017")
+					(reference "J4")
 					(unit 1)
 				)
@@
 	)
 	(symbol
-		(lib_id "Connector_Generic:Conn_01x02")
-		(at 40.64 152.4 0)
+		(lib_id "power:+5V")
+		(at 34.29 148.59 0)
 		(unit 1)
 		(exclude_from_sim no)
@@
 		(on_board yes)
 		(dnp no)
-		(fields_autoplaced yes)
-		(property "Reference" "J12"
-			(at 43.18 152.3999 0)
+		(property "Reference" "#PWR017"
+			(at 34.29 152.4 0)
 			(effects
 				(font
 					(size 1.27 1.27)
 				)
-				(justify left)
+				(hide yes)
 			)
 		)
-		(property "Value" "buzzer"
-			(at 43.18 154.9399 0)
+		(property "Value" "+5V"
+			(at 34.29 143.51 0)
 			(effects
 				(font
 					(size 1.27 1.27)
 				)
-				(justify left)
 			)
 		)
-		(property "Footprint" "Connector_AMASS:AMASS_XT30PW-M_1x02_P2.50mm_Horizontal"
-			(at 40.64 152.4 0)
+		(property "Footprint" ""
+			(at 34.29 148.59 0)
 			(effects
 				(font
@@
 			)
 		)
-		(property "Datasheet" "~"
-			(at 40.64 152.4 0)
+		(property "Datasheet" ""
+			(at 34.29 148.59 0)
 			(effects
 				(font
@@
 			)
 		)
-		(property "Description" "Generic connector, single row, 01x02, script generated (kicad-library-utils/schlib/autogen/connector/)"
-			(at 40.64 152.4 0)
+		(property "Description" "Power symbol creates a global label with name \"+5V\""
+			(at 34.29 148.59 0)
 			(effects
 				(font
@@
 			)
 		)
-		(pin "2"
-		)
 		(pin "1"
 		)
@@
 			(project "cerradura"
 				(path "/5ec40689-7e61-4c5f-9022-56a5e47f7bec"
-					(reference "J12")
+					(reference "#PWR017")
 					(unit 1)
 				)
@@
 					(unit 1)
 				)
+			)
+		)
+	)
+	(symbol
+		(lib_id "Connector:Screw_Terminal_01x02")
+		(at 40.64 152.4 0)
+		(unit 1)
+		(exclude_from_sim no)
+		(in_bom yes)
+		(on_board yes)
+		(dnp no)
+		(fields_autoplaced yes)
+		(property "Reference" "J14"
+			(at 43.18 152.3999 0)
+			(effects
+				(font
+					(size 1.27 1.27)
+				)
+				(justify left)
+			)
+		)
+		(property "Value" "bornes_buzzer"
+			(at 43.18 154.9399 0)
+			(effects
+				(font
+					(size 1.27 1.27)
+				)
+				(justify left)
+			)
+		)
+		(property "Footprint" "TerminalBlock:TerminalBlock_Altech_AK300-2_P5.00mm"
+			(at 40.64 152.4 0)
+			(effects
+				(font
+					(size 1.27 1.27)
+				)
+				(hide yes)
+			)
+		)
+		(property "Datasheet" "~"
+			(at 40.64 152.4 0)
+			(effects
+				(font
+					(size 1.27 1.27)
+				)
+				(hide yes)
+			)
+		)
+		(property "Description" "Generic screw terminal, single row, 01x02, script generated (kicad-library-utils/schlib/autogen/connector/)"
+			(at 40.64 152.4 0)
+			(effects
+				(font
+					(size 1.27 1.27)
+				)
+				(hide yes)
+			)
+		)
+		(pin "1"
+		)
+		(pin "2"
+		)
+		(instances
+			(project ""
+				(path "/5ec40689-7e61-4c5f-9022-56a5e47f7bec"
+					(reference "J14")
+					(unit 1)
+				)

Commit message: cambios dispositivos
Parts:
- removed J10: drv882x_righ_socket, Connector_Harwin:Harwin_M20-89008xx_1x08_P2.54mm_Horizontal, symbol Connector:Conn_01x08_Socket
- removed J3: esp32_c3_right_socket, Connector_Harwin:Harwin_M20-89008xx_1x08_P2.54mm_Horizontal, symbol Connector:Conn_01x08_Socket
- removed J5: esp32_c3_left_socket, Connector_Harwin:Harwin_M20-89008xx_1x08_P2.54mm_Horizontal, symbol Connector:Conn_01x08_Socket
- removed J9: drv882x_left_socket, Connector_Harwin:Harwin_M20-89008xx_1x08_P2.54mm_Horizontal, symbol Connector:Conn_01x08_Socket
- added A1: DRV8825, Module:Pololu_Breakout-16_15.2x20.3mm, symbol Driver_Motor:Pololu_Breakout_DRV8825
- added U1: ESP32_c3_mini, RF_Module:WEMOS_C3_mini, symbol RF_Module:WEMOS_C3_mini
- J11: footprint Connector_Harwin:Harwin_M20-89003xx_1x03_P2.54mm_Horizontal -> Connector_PinHeader_2.54mm:PinHeader_1x03_P2.54mm_Vertical
- J4, J7: footprint Connector_Harwin:Harwin_M20-89008xx_1x08_P2.54mm_Horizontal -> Connector_PinHeader_2.54mm:PinHeader_1x08_P2.54mm_Vertical
- J8: footprint Connector_Harwin:Harwin_M20-89004xx_1x04_P2.54mm_Horizontal -> Connector_PinSocket_2.54mm:PinSocket_1x04_P2.54mm_Vertical
Connections:
- net +3.3V: now also A1.13 (~{RST}), A1.14 (~{SLP}), U1.9 (VBus)
- net GND: now also A1.1 (GND), A1.7 (GND), U1.10 (GND)
- net drv882x_a1: now also A1.4 (A1)
- net drv882x_a2: now also A1.3 (A2)
- net drv882x_b1: now also A1.5 (B1)
- net drv882x_b2: now also A1.6 (B2)
- net drv882x_dir: now also A1.16 (DIR)
- net drv882x_en: now also A1.9 (~{EN})
- net drv882x_step: now also A1.15 (STEP)
- net esp32_rx: now also U1.15 (RX)
- net esp32_tx: now also U1.16 (TX)
