File: esquemasConEdu/cerradura.kicad_sch (KiCad schematic)
At the start: 16 parts, among them Q1 PN2222A

Commit message: jack por bornera
Parts:
- removed 12V-BORN1: Jack-DC, Connector_BarrelJack:BarrelJack_SwitchcraftConxall_RAPC10U_Horizontal, symbol Connector:Jack-DC
- added 12V-BORN: 12V-DC-IN, TerminalBlock:TerminalBlock_Altech_AK300-2_P5.00mm, symbol Connector:Screw_Terminal_01x02
Connections:
- net +12V: now also 12V-BORN.2 (Pin_2)
- net GND: now also 12V-BORN.1 (Pin_1)
Changed lines of the file:
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@@
+	(wire
+		(pts
+			(xy 195.58 95.25) (xy 195.58 97.79)
+		)
+		(stroke
+			(width 0)
+			(type default)
+		)
+	)
 	(wire
 		(pts
@@
 	)
 	(symbol
+		(lib_id "Connector:Screw_Terminal_01x02")
+		(at 190.5 95.25 180)
+		(unit 1)
+		(exclude_from_sim no)
+		(in_bom yes)
+		(on_board yes)
+		(dnp no)
+		(fields_autoplaced yes)
+		(property "Reference" "12V-BORN"
+			(at 190.5 86.36 0)
+			(effects
+				(font
+					(size 1.27 1.27)
+				)
+			)
+		)
+		(property "Value" "12V-DC-IN"
+			(at 190.5 88.9 0)
+			(effects
+				(font
+					(size 1.27 1.27)
+				)
+			)
+		)
+		(property "Footprint" "TerminalBlock:TerminalBlock_Altech_AK300-2_P5.00mm"
+			(at 190.5 95.25 0)
+			(effects
+				(font
+					(size 1.27 1.27)
+				)
+				(hide yes)
+			)
+		)
+		(property "Datasheet" "~"
+			(at 190.5 95.25 0)
+			(effects
+				(font
+					(size 1.27 1.27)
+				)
+				(hide yes)
+			)
+		)
+		(property "Description" "Generic screw terminal, single row, 01x02, script generated (kicad-library-utils/schlib/autogen/connector/)"
+			(at 190.5 95.25 0)
+			(effects
+				(font
+					(size 1.27 1.27)
+				)
+				(hide yes)
+			)
+		)
+		(pin "1"
+		)
+		(pin "2"
+		)
+		(instances
+			(project "cerradura"
+				(path "/5ec40689-7e61-4c5f-9022-56a5e47f7bec"
+					(reference "12V-BORN")
+					(unit 1)
+				)
+			)
+		)
+	)
+	(symbol
 		(lib_id "Connector_Generic:Conn_02x20_Odd_Even")
 		(at 134.62 76.2 0)
@@
 					(unit 1)
 				)
-			)
-		)
-	)
-	(symbol
-		(lib_id "Connector:Jack-DC")
-		(at 187.96 95.25 0)
-		(unit 1)
-		(exclude_from_sim no)
-		(in_bom yes)
-		(on_board yes)
-		(dnp no)
-		(fields_autoplaced yes)
-		(property "Reference" "12V-BORN1"
-			(at 187.96 86.36 0)
-			(effects
-				(font
-					(size 1.27 1.27)
-				)
-			)
-		)
-		(property "Value" "Jack-DC"
-			(at 187.96 88.9 0)
-			(effects
-				(font
-					(size 1.27 1.27)
-				)
-			)
-		)
-		(property "Footprint" "Connector_BarrelJack:BarrelJack_SwitchcraftConxall_RAPC10U_Horizontal"
-			(at 189.23 96.266 0)
-			(effects
-				(font
-					(size 1.27 1.27)
-				)
-				(hide yes)
-			)
-		)
-		(property "Datasheet" "~"
-			(at 189.23 96.266 0)
-			(effects
-				(font
-					(size 1.27 1.27)
-				)
-				(hide yes)
-			)
-		)
-		(property "Description" "DC Barrel Jack"
-			(at 187.96 95.25 0)
-			(effects
-				(font
-					(size 1.27 1.27)
-				)
-				(hide yes)
-			)
-		)
-		(pin "2"
-		)
-		(pin "1"
-		)
-		(instances
-			(project ""
-				(path "/5ec40689-7e61-4c5f-9022-56a5e47f7bec"
-					(reference "12V-BORN1")
-					(unit 1)
-				)

Commit message: plano de tierra
Parts:
- renumbered 12V-BORN to 12V-BORN1
Changed lines of the file:
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@@
 		(dnp no)
 		(fields_autoplaced yes)
-		(property "Reference" "12V-BORN"
+		(property "Reference" "12V-BORN1"
 			(at 190.5 86.36 0)
 			(effects
@@
 			(project "cerradura"
 				(path "/5ec40689-7e61-4c5f-9022-56a5e47f7bec"
-					(reference "12V-BORN")
+					(reference "12V-BORN1")
 					(unit 1)
 				)

Commit message: todo conectado + algunas vias
Connections:
- net buzzer_sgn: now also EDU_L1.4 (Pin_4); no longer EDU_L1.34 (Pin_34)
- net door_sensor: now also EDU_L1.6 (Pin_6); no longer EDU_L1.36 (Pin_36)
Changed lines of the file:
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@@
+	(wire
+		(pts
+			(xy 96.52 55.88) (xy 93.98 55.88)
+		)
+		(stroke
+			(width 0)
+			(type default)
+		)
+	)
 	(wire
 		(pts
@@
 		(pts
 			(xy 45.72 121.92) (xy 39.37 121.92)
+		)
+		(stroke
+			(width 0)
+			(type default)
+		)
+	)
+	(wire
+		(pts
+			(xy 93.98 58.42) (xy 96.52 58.42)
 		)
 		(stroke
@@
 		)
 	)
+	(label "buzzer_sgn"
+		(at 96.52 55.88 0)
+		(effects
+			(font
+				(size 1.27 1.27)
+			)
+			(justify left bottom)
+		)
+	)
 	(label "kp_f2"
 		(at 104.14 121.92 90)
@@
 		)
 	)
-	(label "door_sensor"
-		(at 93.98 96.52 0)
-		(effects
-			(font
-				(size 1.27 1.27)
-			)
-			(justify left bottom)
-		)
-	)
 	(label "kp_f3"
 		(at 129.54 96.52 180)
@@
 		)
 	)
-	(label "buzzer_sgn"
-		(at 93.98 93.98 0)
-		(effects
-			(font
-				(size 1.27 1.27)
-			)
-			(justify left bottom)
-		)
-	)
 	(label "kp_c1"
 		(at 111.76 121.92 90)
@@
 		(effects
 			(font
+				(size 1.27 1.27)
+			)
+			(justify left bottom)
+		)
+	)
+	(label "door_sensor"
+		(at 96.52 58.42 0)
+		(effects
+			(font

Commit message: 'Todo' conectado 1 mm
Parts:
- A3144: value Bornera Sensor Hall -> A3144
- EDU_L1: value EDU_CIAA_LEFT_SOCKET -> EDU_L
- EDU_R1: value EDU_CIAA_RIGHT_SOCKET -> EDU_R
- ESP1: value ESP32_SOCKET -> ESP
- RC522: value RC522_sensor -> RC522
- T1: renamed from Q1; value PN2222A -> BC547
- renumbered MOTOR_BORN1 to bornes_motor1, Keypad1 to num_keypad1
Changed lines of the file:
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@@
 		(dnp no)
 		(fields_autoplaced yes)
-		(property "Reference" "Q1"
+		(property "Reference" "T1"
 			(at 54.61 176.5299 0)
 			(effects
@@
 			)
 		)
-		(property "Value" "PN2222A"
+		(property "Value" "BC547"
 			(at 54.61 179.0699 0)
 			(effects
@@
 			(project ""
 				(path "/5ec40689-7e61-4c5f-9022-56a5e47f7bec"
-					(reference "Q1")
+					(reference "T1")
 					(unit 1)
 				)
@@
 			)
 		)
-		(property "Value" "EDU_CIAA_RIGHT_SOCKET"
+		(property "Value" "EDU_R"
 			(at 135.89 49.53 0)
 			(effects
@@
 			)
 		)
-		(property "Value" "ESP32_SOCKET"
+		(property "Value" "ESP"
 			(at 210.312 51.562 0)
 			(effects
@@
 			)
 		)
-		(property "Value" "Bornera Sensor Hall"
+		(property "Value" "A3144"
 			(at 29.21 64.77 0)
 			(effects
@@
 		(dnp no)
 		(fields_autoplaced yes)
-		(property "Reference" "MOTOR_BORN1"
+		(property "Reference" "bornes_motor1"
 			(at 255.27 140.9699 0)
 			(effects
@@
 			(project ""
 				(path "/5ec40689-7e61-4c5f-9022-56a5e47f7bec"
-					(reference "MOTOR_BORN1")
+					(reference "bornes_motor1")
 					(unit 1)
 				)
@@
 		(on_board yes)
 		(dnp no)
-		(property "Reference" "Keypad1"
+		(property "Reference" "num_keypad1"
 			(at 107.95 133.35 90)
 			(effects
@@
 			(project ""
 				(path "/5ec40689-7e61-4c5f-9022-56a5e47f7bec"
-					(reference "Keypad1")
+					(reference "num_keypad1")
 					(unit 1)
 				)
@@
 			)
 		)
-		(property "Value" "EDU_CIAA_LEFT_SOCKET"
+		(property "Value" "EDU_L"
 			(at 87.63 49.53 0)
 			(effects
@@
 			)
 		)
-		(property "Value" "RC522_sensor"
+		(property "Value" "RC522"
 			(at 151.13 134.62 90)
 			(effects

Commit message: se agrega modulo de deteccion de presencia y resistencia en base de T1
Parts:
- added HW-416-PIR1: HW-416-PIR, Connector_PinSocket_2.54mm:PinSocket_1x03_P2.54mm_Vertical, symbol Connector:Conn_01x03_Pin
- added R2: R2, Connector_PinHeader_1.00mm:PinHeader_1x02_P1.00mm_Vertical, symbol Device:R
- added R3: R3, Connector_PinHeader_1.00mm:PinHeader_1x02_P1.00mm_Vertical, symbol Device:R
- added T2: BC547, Package_TO_SOT_THT:TO-92_Inline, symbol Transistor_BJT:PN2222A
- R1-10K1: renamed from 10K1; value 10K -> R1 (10k)
Connections:
- net +12V: now also T2.1 (E), T2.3 (C)
- net +5V: now also HW-416-PIR1.3 (Pin_3)
- net GND: now also HW-416-PIR1.1 (Pin_1)
- net buzzer_sgn: now also R2.1; no longer T1.2 (B)
- new net: R2.2, T1.2 (B)
- new net: R3.1, T2.2 (B)
- new net hw-416-sgn: HW-416-PIR1.2 (Pin_2), R3.2

Commit message: sensor de presencia con gpio
Connections:
- net hw-416-sgn: now also EDU_L1.12 (Pin_12)
Changed lines of the file:
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@@
+	(wire
+		(pts
+			(xy 95.25 66.04) (xy 93.98 66.04)
+		)
+		(stroke
+			(width 0)
+			(type default)
+		)
+	)
 	(wire
 		(pts
@@
 		(effects
 			(font
+				(size 1.27 1.27)
+			)
+			(justify left bottom)
+		)
+	)
+	(label "hw-416-sgn"
+		(at 95.25 66.04 0)
+		(effects
+			(font

Commit message: correccion en modulo de deteccion de presencia
Parts:
- added Jump1: Jump1, Connector_PinSocket_2.54mm:PinSocket_1x02_P2.54mm_Vertical, symbol Connector:Conn_01x02_Pin
- added Jump2: Jump2, Connector_PinSocket_2.54mm:PinSocket_1x02_P2.54mm_Vertical, symbol Connector:Conn_01x02_Pin
Connections:
- net +12V: no longer T2.1 (E), T2.3 (C)
- net +5V: no longer HW-416-PIR1.3 (Pin_3)
- net hw-416-sgn: now also Jump2.1 (Pin_1); no longer EDU_L1.12 (Pin_12)
- net +5V-out renamed +5V-out-a
- net +5V-out-a: now also HW-416-PIR1.3 (Pin_3), T2.3 (C), Jump1.1 (Pin_1); no longer 5V_BORN1.1 (Pin_1)
- new net +5V-out-b: 5V_BORN1.1 (Pin_1), Jump1.2 (Pin_2), T2.1 (E)
- new net hw-416-sgn-a: EDU_L1.12 (Pin_12), Jump2.2 (Pin_2)
- no-connect marks 0 -> 60
Other:
- moved on the sheet: 12V-BORN1, 5V_BORN1, ESP1, HW-416-PIR1, R3, T2, lm2596hvs1
